File: minta386.kicad_pcb (KiCad board)
At the start: 4 copper layers, 190.5 x 104.8 mm, 63 parts, among them U1 Spare, U2 Spare, U3 Spare, U4 Spare, U43 74F244, U44 74F240, U45 74F244, U57 74F32, U58 74F240, U59 74F244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

Commit message: slight board chnages for rev 1.0
Parts:
- removed JP1, JP2, JP3, JP4: Conn_01x03_Pin, Connector_PinHeader_2.54mm:PinHeader_1x03_P2.54mm_Vertical
Connections:
- J1 pad 38: ~{CAS} -> ~{CAS_B0}
- J1 pad 40: ~{DWE} -> ~{DWE_B0}
- U43 pad 11: Net-(JP4-Pin_2) -> ~{RAS0B}
- U43 pad 13: Net-(JP4-Pin_2) -> ~{RAS0B}
- U43 pad 15: Net-(JP3-Pin_2) -> ~{RAS1B}
- U43 pad 17: Net-(JP3-Pin_2) -> ~{RAS1B}
- U57 pad 1: ~{CAS_B1} -> ~{CAS_B0}
- U57 pad 10: ~{CAS_B1} -> ~{CAS_B0}
- U57 pad 13: ~{CAS_B1} -> ~{CAS_B0}
- U57 pad 4: ~{CAS_B1} -> ~{CAS_B0}
- U64 pad 6: ~{DWE_B1} -> ~{DWE_B0}
- U64 pad 8: ~{DWE_B1} -> ~{DWE_B0}
Routing:
- net ~{DWE_B0}: track 24.2 -> 326.3 mm, vias 0 -> 2
- net ~{DWE}: track 290.5 -> 0.00 mm, vias 2 -> 0
- net ~{CAS_B0}: track 188.9 -> 328.7 mm, vias 1 -> 4
- net ~{CAS}: track 108.8 -> 0.00 mm, vias 2 -> 0
- net ~{CAS_B1}: track 31.7 -> 0.00 mm
- net Net-(JP4-Pin_2): track 21.1 -> 0.00 mm
- net ~{DWE_B1}: track 16.7 -> 0.00 mm
- net ~{RAS0B}: track 273.8 -> 290.5 mm, vias 0 -> 1
- net Net-(JP3-Pin_2): track 12.6 -> 0.00 mm
- net ~{RAS1B}: track 276.9 -> 286.7 mm, vias 1 -> 2
Other:
- board text added: "Minta Technologies 305-1 Mainboard Memory Board v1.0"
- board text removed: "Minta Technologies 305-1 Mainboard Memory Board v0.01"
