File: minta386.kicad_sch (KiCad schematic)
At the start: 62 parts, among them U1 Spare, U2 Spare, U3 Spare, U4 Spare, U43 74F244, U44 74F240, U45 74F244, U57 74F32, U58 74F240, U59 74F244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

Commit message: slight board chnages for rev 1.0
Parts:
- removed JP1, JP2, JP3, JP4: Conn_01x03_Pin, Connector_PinHeader_2.54mm:PinHeader_1x03_P2.54mm_Vertical, symbol Connector:Conn_01x03_Pin
Connections:
- net ~{CAS_B1} is gone; now on net ~{CAS_B0}: U57.1, U57.10, U57.13, U57.4
- net ~{CAS} is gone; now on net ~{CAS_B0}: J1.38 (~{CAS})
- net ~{DWE_B1} is gone; now on net ~{DWE_B0}: U64.6 (I2a), U64.8 (I3a)
- net ~{DWE} is gone; now on net ~{DWE_B0}: J1.40 (~{DWE})
- net ~{RAS0B}: now also U43.11 (I0b), U43.13 (I1b)
- net ~{RAS1B}: now also U43.15 (I2b), U43.17 (I3b)
- no-connect marks 52 -> 50
